File: PCB Design/Cable_Monitor/simulation.kicad_sch (KiCad schematic)
At the start: 9 parts

Commit message: PCB Layout Update
Parts:
- renumbered R22 to R30, R23 to R31, R24 to R32, R25 to R33
Changed lines of the file:
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@@
   (symbol (lib_id "Device:R") (at 106.68 149.86 90) (unit 1)
     (in_bom no) (on_board no) (dnp no)
-    (property "Reference" "R25" (at 106.68 149.86 90)
+    (property "Reference" "R33" (at 106.68 149.86 90)
       (effects (font (size 1.27 1.27)))
     )
@@
       (project "Cable_Monitor"
         (path "/1f276d59-ad9b-4e70-a842-f3b7e562eb9b/7f77e12f-21a5-46a0-a1f3-68c3015df384"
-          (reference "R25") (unit 1)
+          (reference "R33") (unit 1)
         )
       )
@@
   (symbol (lib_id "power:+5V") (at 63.5 139.7 0) (unit 1)
     (in_bom yes) (on_board yes) (dnp no)
-    (property "Reference" "#PWR053" (at 63.5 143.51 0)
+    (property "Reference" "#PWR058" (at 63.5 143.51 0)
       (effects (font (size 1.27 1.27)) hide)
     )
@@
       (project "Cable_Monitor"
         (path "/1f276d59-ad9b-4e70-a842-f3b7e562eb9b/7f77e12f-21a5-46a0-a1f3-68c3015df384"
-          (reference "#PWR053") (unit 1)
+          (reference "#PWR058") (unit 1)
         )
       )
@@
   (symbol (lib_id "Device:R") (at 106.68 147.32 90) (unit 1)
     (in_bom no) (on_board no) (dnp no)
-    (property "Reference" "R24" (at 106.68 147.32 90)
+    (property "Reference" "R32" (at 106.68 147.32 90)
       (effects (font (size 1.27 1.27)))
     )
@@
       (project "Cable_Monitor"
         (path "/1f276d59-ad9b-4e70-a842-f3b7e562eb9b/7f77e12f-21a5-46a0-a1f3-68c3015df384"
-          (reference "R24") (unit 1)
+          (reference "R32") (unit 1)
         )
       )
@@
   (symbol (lib_id "power:GND") (at 63.5 177.8 0) (unit 1)
     (in_bom yes) (on_board yes) (dnp no) (fields_autoplaced)
-    (property "Reference" "#PWR056" (at 63.5 184.15 0)
+    (property "Reference" "#PWR059" (at 63.5 184.15 0)
       (effects (font (size 1.27 1.27)) hide)
     )
@@
       (project "Cable_Monitor"
         (path "/1f276d59-ad9b-4e70-a842-f3b7e562eb9b/7f77e12f-21a5-46a0-a1f3-68c3015df384"
-          (reference "#PWR056") (unit 1)
+          (reference "#PWR059") (unit 1)
         )
       )
@@
   (symbol (lib_id "power:GND") (at 152.4 177.8 0) (unit 1)
     (in_bom yes) (on_board yes) (dnp no) (fields_autoplaced)
-    (property "Reference" "#PWR023" (at 152.4 184.15 0)
+    (property "Reference" "#PWR061" (at 152.4 184.15 0)
       (effects (font (size 1.27 1.27)) hide)
     )
@@
       (project "Cable_Monitor"
         (path "/1f276d59-ad9b-4e70-a842-f3b7e562eb9b/7f77e12f-21a5-46a0-a1f3-68c3015df384"
-          (reference "#PWR023") (unit 1)
+          (reference "#PWR061") (unit 1)
         )
       )
@@
   (symbol (lib_id "Device:R") (at 106.68 144.78 90) (unit 1)
     (in_bom no) (on_board no) (dnp no)
-    (property "Reference" "R23" (at 106.68 144.78 90)
+    (property "Reference" "R31" (at 106.68 144.78 90)
       (effects (font (size 1.27 1.27)))
     )
@@
       (project "Cable_Monitor"
         (path "/1f276d59-ad9b-4e70-a842-f3b7e562eb9b/7f77e12f-21a5-46a0-a1f3-68c3015df384"
-          (reference "R23") (unit 1)
+          (reference "R31") (unit 1)
         )
       )
@@
   (symbol (lib_id "power:GND") (at 101.6 177.8 0) (unit 1)
     (in_bom yes) (on_board yes) (dnp no) (fields_autoplaced)
-    (property "Reference" "#PWR055" (at 101.6 184.15 0)
+    (property "Reference" "#PWR060" (at 101.6 184.15 0)
       (effects (font (size 1.27 1.27)) hide)
     )
@@
       (project "Cable_Monitor"
         (path "/1f276d59-ad9b-4e70-a842-f3b7e562eb9b/7f77e12f-21a5-46a0-a1f3-68c3015df384"
-          (reference "#PWR055") (unit 1)
+          (reference "#PWR060") (unit 1)
         )
       )
@@
   (symbol (lib_id "power:+3V0") (at 38.1 139.7 0) (unit 1)
     (in_bom yes) (on_board yes) (dnp no)
-    (property "Reference" "#PWR052" (at 38.1 143.51 0)
+    (property "Reference" "#PWR056" (at 38.1 143.51 0)
       (effects (font (size 1.27 1.27)) hide)
     )
@@
       (project "Cable_Monitor"
         (path "/1f276d59-ad9b-4e70-a842-f3b7e562eb9b/7f77e12f-21a5-46a0-a1f3-68c3015df384"
-          (reference "#PWR052") (unit 1)
+          (reference "#PWR056") (unit 1)
         )
       )
@@
   (symbol (lib_id "Device:R") (at 106.68 142.24 90) (unit 1)
     (in_bom no) (on_board no) (dnp no)
-    (property "Reference" "R22" (at 106.68 142.24 90)
+    (property "Reference" "R30" (at 106.68 142.24 90)
       (effects (font (size 1.27 1.27)))
     )
@@
       (project "Cable_Monitor"
         (path "/1f276d59-ad9b-4e70-a842-f3b7e562eb9b/7f77e12f-21a5-46a0-a1f3-68c3015df384"
-          (reference "R22") (unit 1)
-        )
-      )
+          (reference "R30") (unit 1)
+        )
+      )

Commit message: PCB Design Update
Parts:
- renumbered R30 to R28, R31 to R29, R32 to R30, R33 to R31
Changed lines of the file:
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@@
   (symbol (lib_id "Device:R") (at 106.68 149.86 90) (unit 1)
     (in_bom no) (on_board no) (dnp no)
-    (property "Reference" "R33" (at 106.68 149.86 90)
+    (property "Reference" "R31" (at 106.68 149.86 90)
       (effects (font (size 1.27 1.27)))
     )
@@
       (project "Cable_Monitor"
         (path "/1f276d59-ad9b-4e70-a842-f3b7e562eb9b/7f77e12f-21a5-46a0-a1f3-68c3015df384"
-          (reference "R33") (unit 1)
+          (reference "R31") (unit 1)
         )
       )
@@
   (symbol (lib_id "power:+5V") (at 63.5 139.7 0) (unit 1)
     (in_bom yes) (on_board yes) (dnp no)
-    (property "Reference" "#PWR058" (at 63.5 143.51 0)
+    (property "Reference" "#PWR062" (at 63.5 143.51 0)
       (effects (font (size 1.27 1.27)) hide)
     )
@@
       (project "Cable_Monitor"
         (path "/1f276d59-ad9b-4e70-a842-f3b7e562eb9b/7f77e12f-21a5-46a0-a1f3-68c3015df384"
-          (reference "#PWR058") (unit 1)
+          (reference "#PWR062") (unit 1)
         )
       )
@@
   (symbol (lib_id "Device:R") (at 106.68 147.32 90) (unit 1)
     (in_bom no) (on_board no) (dnp no)
-    (property "Reference" "R32" (at 106.68 147.32 90)
+    (property "Reference" "R30" (at 106.68 147.32 90)
       (effects (font (size 1.27 1.27)))
     )
@@
       (project "Cable_Monitor"
         (path "/1f276d59-ad9b-4e70-a842-f3b7e562eb9b/7f77e12f-21a5-46a0-a1f3-68c3015df384"
-          (reference "R32") (unit 1)
+          (reference "R30") (unit 1)
         )
       )
@@
   (symbol (lib_id "power:GND") (at 63.5 177.8 0) (unit 1)
     (in_bom yes) (on_board yes) (dnp no) (fields_autoplaced)
-    (property "Reference" "#PWR059" (at 63.5 184.15 0)
+    (property "Reference" "#PWR063" (at 63.5 184.15 0)
       (effects (font (size 1.27 1.27)) hide)
     )
@@
       (project "Cable_Monitor"
         (path "/1f276d59-ad9b-4e70-a842-f3b7e562eb9b/7f77e12f-21a5-46a0-a1f3-68c3015df384"
-          (reference "#PWR059") (unit 1)
+          (reference "#PWR063") (unit 1)
         )
       )
@@
   (symbol (lib_id "power:GND") (at 152.4 177.8 0) (unit 1)
     (in_bom yes) (on_board yes) (dnp no) (fields_autoplaced)
-    (property "Reference" "#PWR061" (at 152.4 184.15 0)
+    (property "Reference" "#PWR065" (at 152.4 184.15 0)
       (effects (font (size 1.27 1.27)) hide)
     )
@@
       (project "Cable_Monitor"
         (path "/1f276d59-ad9b-4e70-a842-f3b7e562eb9b/7f77e12f-21a5-46a0-a1f3-68c3015df384"
-          (reference "#PWR061") (unit 1)
+          (reference "#PWR065") (unit 1)
         )
       )
@@
   (symbol (lib_id "power:GND") (at 38.1 177.8 0) (unit 1)
     (in_bom yes) (on_board yes) (dnp no) (fields_autoplaced)
-    (property "Reference" "#PWR057" (at 38.1 184.15 0)
+    (property "Reference" "#PWR061" (at 38.1 184.15 0)
       (effects (font (size 1.27 1.27)) hide)
     )
@@
       (project "Cable_Monitor"
         (path "/1f276d59-ad9b-4e70-a842-f3b7e562eb9b/7f77e12f-21a5-46a0-a1f3-68c3015df384"
-          (reference "#PWR057") (unit 1)
+          (reference "#PWR061") (unit 1)
         )
       )
@@
   (symbol (lib_id "Device:R") (at 106.68 144.78 90) (unit 1)
     (in_bom no) (on_board no) (dnp no)
-    (property "Reference" "R31" (at 106.68 144.78 90)
+    (property "Reference" "R29" (at 106.68 144.78 90)
       (effects (font (size 1.27 1.27)))
     )
@@
       (project "Cable_Monitor"
         (path "/1f276d59-ad9b-4e70-a842-f3b7e562eb9b/7f77e12f-21a5-46a0-a1f3-68c3015df384"
-          (reference "R31") (unit 1)
+          (reference "R29") (unit 1)
         )
       )
@@
   (symbol (lib_id "power:GND") (at 101.6 177.8 0) (unit 1)
     (in_bom yes) (on_board yes) (dnp no) (fields_autoplaced)
-    (property "Reference" "#PWR060" (at 101.6 184.15 0)
+    (property "Reference" "#PWR064" (at 101.6 184.15 0)
       (effects (font (size 1.27 1.27)) hide)
     )
@@
       (project "Cable_Monitor"
         (path "/1f276d59-ad9b-4e70-a842-f3b7e562eb9b/7f77e12f-21a5-46a0-a1f3-68c3015df384"
-          (reference "#PWR060") (unit 1)
+          (reference "#PWR064") (unit 1)
         )
       )
@@
   (symbol (lib_id "power:+3V0") (at 38.1 139.7 0) (unit 1)
     (in_bom yes) (on_board yes) (dnp no)
-    (property "Reference" "#PWR056" (at 38.1 143.51 0)
+    (property "Reference" "#PWR060" (at 38.1 143.51 0)
       (effects (font (size 1.27 1.27)) hide)
     )
@@
       (project "Cable_Monitor"
         (path "/1f276d59-ad9b-4e70-a842-f3b7e562eb9b/7f77e12f-21a5-46a0-a1f3-68c3015df384"
-          (reference "#PWR056") (unit 1)
+          (reference "#PWR060") (unit 1)
         )
       )
@@
   (symbol (lib_id "Device:R") (at 106.68 142.24 90) (unit 1)
     (in_bom no) (on_board no) (dnp no)
-    (property "Reference" "R30" (at 106.68 142.24 90)
+    (property "Reference" "R28" (at 106.68 142.24 90)
       (effects (font (size 1.27 1.27)))
     )
@@
       (project "Cable_Monitor"
         (path "/1f276d59-ad9b-4e70-a842-f3b7e562eb9b/7f77e12f-21a5-46a0-a1f3-68c3015df384"
-          (reference "R30") (unit 1)
-        )
-      )
+          (reference "R28") (unit 1)
+        )
+      )
