File: PCB Design/Cable_Monitor/miscellaneous.kicad_sch (KiCad schematic)
At the start: 28 parts, among them J1 ${SIM.PARAMS}, Q1 BSS316N, SW1 ${SIM.PARAMS}, U3 SiP32508, U4 LD1117S33TR_SOT223, U5 ${SIM.PARAMS}, U6 ${SIM.PARAMS}, Y1 ${SIM.PARAMS}, Y2 ${SIM.PARAMS}

Commit message: PCB Layout Update
Parts:
- removed C4: 100uF, Capacitor_SMD:C_1206_3216Metric_Pad1.33x1.80mm_HandSolder, symbol Device:C
- removed C6, C7: 10uF, Capacitor_SMD:C_0805_2012Metric_Pad1.18x1.45mm_HandSolder, symbol Device:C
- removed J1: ${SIM.PARAMS}, Connector_USB:USB_Mini-B_Lumberg_2486_01_Horizontal, symbol Connector:USB_B_Mini
- removed R13, R17: 1k, Resistor_SMD:R_0805_2012Metric_Pad1.20x1.40mm_HandSolder, symbol Device:R
- removed U3: SiP32508, Package_TO_SOT_SMD:TSOT-23-6_HandSoldering, symbol HW_template:SiP32508
- removed U4: LD1117S33TR_SOT223, Package_TO_SOT_SMD:SOT-223-3_TabPin2, symbol Regulator_Linear:LD1117S33TR_SOT223
- renumbered C8 to C18, C9 to C19, R9 to R23, R10 to R24, R11 to R25, R12 to R26, R14 to R27, R15 to R28, R16 to R29, U5 to U7, U6 to U8
Other:
- note removed: "Linear 3.3V low drop regulator The 3V from the microcontroller board can also be used or the microcontroller can be feed by this regulator. Connect to correct supply nets or header pins."
- note removed: "Load switch Can be used to power on with pushbutton and power off via microcontroller. Connect to correct supply nets or header pins."
- note removed: "USB connector might be useful for additional external supply"

Commit message: PCB Design Update
Parts:
- R21: renamed from R23; value 22 -> 65
- renumbered C18 to C24, C19 to C25, R24 to R22, R25 to R23, R26 to R24, R27 to R25, R28 to R26, R29 to R27, U7 to U8, U8 to U9

Commit message: Letzte Anpassungen am Schema
Parts:
- renumbered LED1 to LED3, LED2 to LED4, LED3 to LED5, Q1 to Q2, R21 to R24, R22 to R25, R23 to R26, R24 to R27, R25 to R28, R26 to R29, R27 to R30, SW1 to SW2
