File: PCB Design/Cable_Monitor/Cable_Monitor.kicad_pcb (KiCad board)
At the start: 2 copper layers, 63.5 x 118.1 mm, 85 parts, among them J1 USB_B_Micro, P1 type="R" model="Conn_01x32_Fe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, P2 type="R" model="Conn_01x32_Fe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, Q1 BSS316N, SW1 type="R" model="SW_Push" lib=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, U1 SiP32508, U2 LD1117S33TR, U3 DRV5053_THT, U4 DRV5053_THT, U5 MCP6002-xSN, U6 MCP6002-xSN, U7 MCP6002-xSN

Commit message: a
Parts:
- moved U5 86.5 mm to (147.3, 54.6)
- moved U7 78.9 mm to (135.9, 62.2)
- moved TP10 42.5 mm to (99.1, 162.6)
- moved TP14 28.3 mm to (88.9, 116.8)
- moved U6 22.9 mm to (124.5, 54.6)
- moved TP12 21.1 mm to (71.1, 119.4)
- moved TP17 9.71 mm to (161.3, 158.8)
- moved TP8 9.55 mm to (48.3, 140.3)
- moved TP22 2.54 mm to (86.4, 144.8)
Changed lines of the file:
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@@
   (net 93 "Net-(R20-Pad1)")
   (footprint "TestPoint:TestPoint_Loop_D2.60mm_Drill1.6mm_Beaded" (layer "F.Cu")
-    (at 72.9625 140.28)
+    (at 88.9 116.84)
     (descr "wire loop with bead as test point, loop diameter2.6mm, hole diameter 1.6mm")
     (tags "test point wire loop bead")
@@
         (effects (font (size 1 1) (thickness 0.15)))
     )
-    (fp_text value "3V" (at 0 -2.8) (layer "F.Fab")
+    (fp_text value "3V" (at 0 -2.8) (layer "F.SilkS")
         (effects (font (size 1 1) (thickness 0.15)))
     )
@@
   )
   (footprint "Package_SO:SOIC-8_3.9x4.9mm_P1.27mm" (layer "F.Cu")
-    (at 60.868 55.753)
+    (at 147.32 54.61)
     (descr "SOIC, 8 Pin (JEDEC MS-012AA, https://www.analog.com/media/en/package-pcb-resources/package/pkg_pdf/soic_narrow-r/r_8.pdf), generated with kicad-footprint-generator ipc_gullwing_generator.py")
     (tags "SOIC SO")
@@
   )
   (footprint "Package_SO:SOIC-8_3.9x4.9mm_P1.27mm" (layer "F.Cu")
-    (at 118.4425 76.708)
+    (at 124.46 54.61)
     (descr "SOIC, 8 Pin (JEDEC MS-012AA, https://www.analog.com/media/en/package-pcb-resources/package/pkg_pdf/soic_narrow-r/r_8.pdf), generated with kicad-footprint-generator ipc_gullwing_generator.py")
     (tags "SOIC SO")
@@
   )
   (footprint "TestPoint:TestPoint_Loop_D2.60mm_Drill1.6mm_Beaded" (layer "F.Cu")
-    (at 67.9125 140.28)
+    (at 71.12 119.38)
     (descr "wire loop with bead as test point, loop diameter2.6mm, hole diameter 1.6mm")
     (tags "test point wire loop bead")
@@
         (effects (font (size 1 1) (thickness 0.15)))
     )
-    (fp_text value "pad_left_out" (at 0 -2.8) (layer "F.Fab")
+    (fp_text value "pad_left_out" (at 0 -2.8) (layer "F.SilkS")
         (effects (font (size 1 1) (thickness 0.15)))
     )
@@
         (effects (font (size 1 1) (thickness 0.15)))
     )
-    (fp_text value "pad_right_out" (at 0 -2.8) (layer "F.Fab")
+    (fp_text value "pad_right_out" (at 0 -2.8) (layer "F.SilkS")
         (effects (font (size 1 1) (thickness 0.15)))
     )
@@
         (effects (font (size 1 1) (thickness 0.15)))
     )
-    (fp_text value "pad_left_in" (at 0 -2.8) (layer "F.Fab")
+    (fp_text value "pad_left_in" (at 0 -2.8) (layer "F.SilkS")
         (effects (font (size 1 1) (thickness 0.15)))
     )
@@
   )
   (footprint "TestPoint:TestPoint_Loop_D2.60mm_Drill1.6mm_Beaded" (layer "F.Cu")
-    (at 62.8625 140.28)
+    (at 99.06 162.56)
     (descr "wire loop with bead as test point, loop diameter2.6mm, hole diameter 1.6mm")
     (tags "test point wire loop bead")
@@
         (effects (font (size 1 1) (thickness 0.15)))
     )
-    (fp_text value "pad_left_in" (at 0 -2.8) (layer "F.Fab")
+    (fp_text value "pad_left_in" (at 0 -2.8) (layer "F.SilkS")
         (effects (font (size 1 1) (thickness 0.15)))
     )
@@
         (effects (font (size 1 1) (thickness 0.15)))
     )
-    (fp_text value "5V" (at 0 -2.8) (layer "F.Fab")
+    (fp_text value "5V" (at 0 -2.8) (layer "F.SilkS")
         (effects (font (size 1 1) (thickness 0.15)))
     )
@@
   )
   (footprint "TestPoint:TestPoint_Loop_D2.60mm_Drill1.6mm_Beaded" (layer "F.Cu")
-    (at 86.36 142.24)
+    (at 86.36 144.78)
     (descr "wire loop with bead as test point, loop diameter2.6mm, hole diameter 1.6mm")
     (tags "test point wire loop bead")
@@
         (effects (font (size 1 1) (thickness 0.15)))
     )
-    (fp_text value "HS_right_VGND" (at 0 -2.8) (layer "F.Fab")
+    (fp_text value "HS_right_VGND" (at 0 -2.8) (layer "F.SilkS")
         (effects (font (size 1 1) (thickness 0.15)))
     )
@@
         (effects (font (size 1 1) (thickness 0.15)))
     )
-    (fp_text value "HS_left_VGND" (at 0 -2.8) (layer "F.Fab")
+    (fp_text value "HS_left_VGND" (at 0 -2.8) (layer "F.SilkS")
         (effects (font (size 1 1) (thickness 0.15)))
     )
@@
         (effects (font (size 1 1) (thickness 0.15)))
     )
-    (fp_text value "GND" (at 0 -2.8) (layer "F.Fab")
+    (fp_text value "GND" (at 0 -2.8) (layer "F.SilkS")
         (effects (font (size 1 1) (thickness 0.15)))
     )
@@
   )
   (footprint "TestPoint:TestPoint_Loop_D2.60mm_Drill1.6mm_Beaded" (layer "F.Cu")
-    (at 57.8125 140.28)
+    (at 48.26 140.28)
     (descr "wire loop with bead as test point, loop diameter2.6mm, hole diameter 1.6mm")
     (tags "test point wire loop bead")
@@
         (effects (font (size 1 1) (thickness 0.15)))
     )
-    (fp_text value "Virtual Ground TP" (at 0 -2.8) (layer "F.Fab")
+    (fp_text value "Virtual Ground TP" (at 0 -2.8) (layer "F.SilkS")
         (effects (font (size 1 1) (thickness 0.15)))
     )
@@
   )
   (footprint "TestPoint:TestPoint_Loop_D2.60mm_Drill1.6mm_Beaded" (layer "F.Cu")
-    (at 152.4 162.65)
+    (at 161.29 158.75)
     (descr "wire loop with bead as test point, loop diameter2.6mm, hole diameter 1.6mm")
     (tags "test point wire loop bead")
@@
   )
   (footprint "Package_SO:SOIC-8_3.9x4.9mm_P1.27mm" (layer "F.Cu")
-    (at 211.61 40.17)
+    (at 135.89 62.23)
     (descr "SOIC, 8 Pin (JEDEC MS-012AA, https://www.analog.com/media/en/package-pcb-resources/package/pkg_pdf/soic_narrow-r/r_8.pdf), generated with kicad-footprint-generator ipc_gullwing_generator.py")
     (tags "SOIC SO")

Commit message: Update
Parts:
- removed Lconn1, Lconn2: Conn_01x02_Male, Connector_PinHeader_2.54mm:PinHeader_1x02_P2.54mm_Vertical
- added D1: D, Diode_SMD:D_0805_2012Metric_Pad1.15x1.40mm_HandSolder, F.Cu at (84.1, 82.4)
- added D2: D, Diode_SMD:D_0805_2012Metric_Pad1.15x1.40mm_HandSolder, F.Cu at (89.0, 82.4)
- added HS_Left1: Conn_01x02_Male, Connector_PinHeader_2.54mm:PinHeader_1x02_P2.54mm_Vertical, F.Cu at (132.7, 50.2)
- added HS_right1: Conn_01x02_Male, Connector_PinHeader_2.54mm:PinHeader_1x02_P2.54mm_Vertical, F.Cu at (139.1, 50.2)
- added R24: 1k, Resistor_SMD:R_0805_2012Metric_Pad1.20x1.40mm_HandSolder, F.Cu at (76.4, 31.7)
- added R25: 10k, Resistor_SMD:R_0805_2012Metric_Pad1.20x1.40mm_HandSolder, F.Cu at (76.4, 34.7)
- added R26: 10k, Resistor_SMD:R_0805_2012Metric_Pad1.20x1.40mm_HandSolder, F.Cu at (76.4, 37.6)
- J1: footprint Connector_USB:USB_Micro-B_Molex_47346-0001 -> Connector_USB:USB_Micro-B_Molex-105017-0001
- R10: value 7.5k -> 1M
- R11: value 7.5k -> 5.1k
- R12: value 560k -> 5.1k
- R13: value 560k -> 7.5k
- R14: value 10k -> 7.5k
- R15: value 10k -> 560k
- R16: value 100k -> 560k
- R17: value 100k -> 10k
- R18: value 1M -> 10k
- R19: value 1k -> 100k
- R20: value 1M -> 100k
- R21: value 1k -> 1M
- R22: value 10k -> 1k
- R23: value 10k -> 1M
- R4: value 62 -> 10k
- R5: value 62 -> 30k
- R6: value 1M -> 43k
- R7: value 1M -> 62
- R8: value 5.1k -> 62
- R9: value 5.1k -> 1M
- SW1: value type="R" model="SW_Push" lib="" -> On / Off Button
- TP7: value PWM_Buzzer -> VGND
- TP8: value Virtual Ground TP -> PWM_Buzzer
- moved TP8 139.4 mm to (181.0, 97.8)
- moved TP16 134.5 mm to (153.0, 55.9)
- moved R3 127.3 mm to (185.3, 97.9), turned to -90 degrees
- moved R4 118.0 mm to (88.1, 85.7), turned to 90 degrees
- moved TP15 111.2 mm to (118.7, 55.9)
- moved LED2 98.5 mm to (165.1, 59.7)
- moved Q1 94.6 mm to (189.7, 97.9)
- moved C7 87.8 mm to (134.5, 41.0), turned to 90 degrees
- moved LED1 70.1 mm to (106.7, 59.7)
- moved C8 45.7 mm to (137.4, 42.8), turned to -90 degrees
- moved BZ1 44.6 mm to (182.9, 88.3)
- moved R6 31.9 mm to (94.1, 85.7), turned to 90 degrees
- moved R5 31.2 mm to (93.2, 82.4)
- moved TP7 13.0 mm to (190.1, 69.1)
- moved U5 10.2 mm to (148.6, 64.8)
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Connections:
- R10 pad 1: Net-(C11-Pad1) -> pad_left
- R10 pad 2: GND -> VGND
- R11 pad 1: Net-(C13-Pad1) -> Net-(U6A--)
- R11 pad 2: GND -> Net-(C13-Pad1)
- R12 pad 1: PF6 -> Net-(U5A--)
- R12 pad 2: Net-(U5B--) -> Net-(C11-Pad1)
- R13 pad 1: PC3 -> Net-(C11-Pad1)
- R13 pad 2: Net-(U6B--) -> GND
- R14 pad 1: /hall-sensor_left_right/in_left -> Net-(C13-Pad1)
- R14 pad 2: Net-(C16-Pad2) -> GND
- R15 pad 1: /hall-sensor_left_right/in_right -> PF6
- R15 pad 2: Net-(C17-Pad2) -> Net-(U5B--)
- R16 pad 1: Net-(U7A-+) -> PC3
- R16 pad 2: VGND -> Net-(U6B--)
- R17 pad 1: Net-(U7B-+) -> /hall-sensor_left_right/in_left
- R17 pad 2: VGND -> Net-(C16-Pad2)
- R18 pad 1: Net-(R18-Pad1) -> /hall-sensor_left_right/in_right
- R18 pad 2: Net-(U7A--) -> Net-(C17-Pad2)
- R19 pad 1: Net-(U7A--) -> Net-(U7A-+)
- R19 pad 2: Net-(C20-Pad1) -> VGND
- R20 pad 1: Net-(R20-Pad1) -> Net-(U7B-+)
- R20 pad 2: Net-(U7B--) -> VGND
- R21 pad 1: Net-(U7B--) -> Net-(R21-Pad1)
- R21 pad 2: Net-(C21-Pad1) -> Net-(U7A--)
- R22 pad 1: Net-(R18-Pad1) -> Net-(U7A--)
- R22 pad 2: PF8_ -> Net-(C20-Pad1)
- R23 pad 1: Net-(R20-Pad1) -> Net-(R23-Pad1)
- R23 pad 2: PC1_ -> Net-(U7B--)
- R4 pad 1: PE15_ -> GND
- R4 pad 2: Net-(LED1-A) -> Enable
- R5 pad 1: PE13_ -> Net-(D2-A)
- R5 pad 2: Net-(LED2-A) -> PE3
- R6 pad 1: pad_right -> GND
- R6 pad 2: VGND -> PE3
- R7 pad 1: pad_left -> PE15_
- R7 pad 2: VGND -> Net-(LED1-A)
- R8 pad 1: Net-(U6A--) -> PE13_
- R8 pad 2: Net-(C13-Pad1) -> Net-(LED2-A)
- R9 pad 1: Net-(U5A--) -> pad_right
- R9 pad 2: Net-(C11-Pad1) -> VGND
- SW1 pad 1: unconnected-(SW1-Pad1) -> Net-(D2-A)
- SW1 pad 2: unconnected-(SW1-Pad2) -> +5V
- TP7 pad 1: PA5 -> VGND
- TP8 pad 1: VGND -> PA5
- U7 pad 1: Net-(R18-Pad1) -> Net-(R21-Pad1)
- U7 pad 7: Net-(R20-Pad1) -> Net-(R23-Pad1)
