File: PCB Design/Cable_Monitor/amplifier_filter_1channel.kicad_sch (KiCad schematic)
At the start: 22 parts, among them U7 MCP6002-xSN

Commit message: Updated Schematics
Parts:
- renumbered C15 to C16, C16 to C17, C17 to C18, C18 to C19, C19 to C20, C20 to C21, C21 to C22, C22 to C23, C23 to C24
Changed lines of the file:
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@@
   (symbol (lib_id "Device:C") (at 154.94 76.835 0) (unit 1)
     (in_bom yes) (on_board yes) (dnp no) (fields_autoplaced)
-    (property "Reference" "C20" (at 158.75 75.565 0)
+    (property "Reference" "C21" (at 158.75 75.565 0)
       (effects (font (size 1.27 1.27)) (justify left))
     )
@@
       (project "Cable_Monitor"
         (path "/1f276d59-ad9b-4e70-a842-f3b7e562eb9b/de01ffac-1f9d-4a03-9ae5-48822ed64956"
-          (reference "C20") (unit 1)
+          (reference "C21") (unit 1)
         )
       )
@@
   (symbol (lib_id "Device:C") (at 180.975 114.3 0) (unit 1)
     (in_bom yes) (on_board yes) (dnp no) (fields_autoplaced)
-    (property "Reference" "C23" (at 184.785 113.03 0)
+    (property "Reference" "C24" (at 184.785 113.03 0)
       (effects (font (size 1.27 1.27)) (justify left))
     )
@@
       (project "Cable_Monitor"
         (path "/1f276d59-ad9b-4e70-a842-f3b7e562eb9b/de01ffac-1f9d-4a03-9ae5-48822ed64956"
-          (reference "C23") (unit 1)
+          (reference "C24") (unit 1)
         )
       )
@@
   (symbol (lib_id "power:GND") (at 180.975 122.555 0) (unit 1)
     (in_bom yes) (on_board yes) (dnp no) (fields_autoplaced)
-    (property "Reference" "#PWR049" (at 180.975 128.905 0)
+    (property "Reference" "#PWR050" (at 180.975 128.905 0)
       (effects (font (size 1.27 1.27)) hide)
     )
@@
       (project "Cable_Monitor"
         (path "/1f276d59-ad9b-4e70-a842-f3b7e562eb9b/de01ffac-1f9d-4a03-9ae5-48822ed64956"
-          (reference "#PWR049") (unit 1)
+          (reference "#PWR050") (unit 1)
         )
       )
@@
   (symbol (lib_id "power:GND") (at 155.575 137.16 0) (unit 1)
     (in_bom yes) (on_board yes) (dnp no) (fields_autoplaced)
-    (property "Reference" "#PWR047" (at 155.575 143.51 0)
+    (property "Reference" "#PWR048" (at 155.575 143.51 0)
       (effects (font (size 1.27 1.27)) hide)
     )
@@
       (project "Cable_Monitor"
         (path "/1f276d59-ad9b-4e70-a842-f3b7e562eb9b/de01ffac-1f9d-4a03-9ae5-48822ed64956"
-          (reference "#PWR047") (unit 1)
+          (reference "#PWR048") (unit 1)
         )
       )
@@
   (symbol (lib_id "Device:C") (at 90.17 57.15 180) (unit 1)
     (in_bom yes) (on_board yes) (dnp no) (fields_autoplaced)
-    (property "Reference" "C16" (at 93.98 55.88 0)
+    (property "Reference" "C17" (at 93.98 55.88 0)
       (effects (font (size 1.27 1.27)) (justify right))
     )
@@
       (project "Cable_Monitor"
         (path "/1f276d59-ad9b-4e70-a842-f3b7e562eb9b/de01ffac-1f9d-4a03-9ae5-48822ed64956"
-          (reference "C16") (unit 1)
+          (reference "C17") (unit 1)
         )
       )
@@
   (symbol (lib_id "Device:C") (at 180.34 58.42 0) (unit 1)
     (in_bom yes) (on_board yes) (dnp no) (fields_autoplaced)
-    (property "Reference" "C22" (at 184.15 57.15 0)
+    (property "Reference" "C23" (at 184.15 57.15 0)
       (effects (font (size 1.27 1.27)) (justify left))
     )
@@
       (project "Cable_Monitor"
         (path "/1f276d59-ad9b-4e70-a842-f3b7e562eb9b/de01ffac-1f9d-4a03-9ae5-48822ed64956"
-          (reference "C22") (unit 1)
+          (reference "C23") (unit 1)
         )
       )
@@
   (symbol (lib_id "Device:C") (at 102.87 50.8 90) (unit 1)
     (in_bom yes) (on_board yes) (dnp no) (fields_autoplaced)
-    (property "Reference" "C18" (at 102.87 43.18 90)
+    (property "Reference" "C19" (at 102.87 43.18 90)
       (effects (font (size 1.27 1.27)))
     )
@@
       (project "Cable_Monitor"
         (path "/1f276d59-ad9b-4e70-a842-f3b7e562eb9b/de01ffac-1f9d-4a03-9ae5-48822ed64956"
-          (reference "C18") (unit 1)
+          (reference "C19") (unit 1)
         )
       )
@@
   (symbol (lib_id "power:GND") (at 180.34 66.675 0) (unit 1)
     (in_bom yes) (on_board yes) (dnp no) (fields_autoplaced)
-    (property "Reference" "#PWR048" (at 180.34 73.025 0)
+    (property "Reference" "#PWR049" (at 180.34 73.025 0)
       (effects (font (size 1.27 1.27)) hide)
     )
@@
       (project "Cable_Monitor"
         (path "/1f276d59-ad9b-4e70-a842-f3b7e562eb9b/de01ffac-1f9d-4a03-9ae5-48822ed64956"
-          (reference "#PWR048") (unit 1)
+          (reference "#PWR049") (unit 1)
         )
       )
@@
   (symbol (lib_id "Device:C") (at 28.575 167.64 0) (unit 1)
     (in_bom yes) (on_board yes) (dnp no) (fields_autoplaced)
-    (property "Reference" "C15" (at 32.385 166.3699 0)
+    (property "Reference" "C16" (at 32.385 166.3699 0)
       (effects (font (size 1.27 1.27)) (justify left))
     )
@@
       (project "Cable_Monitor"
         (path "/1f276d59-ad9b-4e70-a842-f3b7e562eb9b/de01ffac-1f9d-4a03-9ae5-48822ed64956"
-          (reference "C15") (unit 1)
+          (reference "C16") (unit 1)
         )
       )
@@
   (symbol (lib_id "power:GND") (at 41.275 175.26 0) (unit 1)
     (in_bom yes) (on_board yes) (dnp no) (fields_autoplaced)
-    (property "Reference" "#PWR043" (at 41.275 181.61 0)
+    (property "Reference" "#PWR044" (at 41.275 181.61 0)
       (effects (font (size 1.27 1.27)) hide)
     )
@@
       (project "Cable_Monitor"
         (path "/1f276d59-ad9b-4e70-a842-f3b7e562eb9b/de01ffac-1f9d-4a03-9ae5-48822ed64956"
-          (reference "#PWR043") (unit 1)
+          (reference "#PWR044") (unit 1)
         )
       )
@@
   (symbol (lib_id "Device:C") (at 90.805 113.03 180) (unit 1)
     (in_bom yes) (on_board yes) (dnp no) (fields_autoplaced)
-    (property "Reference" "C17" (at 94.615 111.76 0)
+    (property "Reference" "C18" (at 94.615 111.76 0)
       (effects (font (size 1.27 1.27)) (justify right))
     )
@@
       (project "Cable_Monitor"
         (path "/1f276d59-ad9b-4e70-a842-f3b7e562eb9b/de01ffac-1f9d-4a03-9ae5-48822ed64956"
-          (reference "C17") (unit 1)
+          (reference "C18") (unit 1)
         )
       )
@@
   (symbol (lib_id "power:GND") (at 154.94 81.28 0) (unit 1)
     (in_bom yes) (on_board yes) (dnp no) (fields_autoplaced)
-    (property "Reference" "#PWR046" (at 154.94 87.63 0)
+    (property "Reference" "#PWR047" (at 154.94 87.63 0)
       (effects (font (size 1.27 1.27)) hide)
     )
@@
       (project "Cable_Monitor"
         (path "/1f276d59-ad9b-4e70-a842-f3b7e562eb9b/de01ffac-1f9d-4a03-9ae5-48822ed64956"
-          (reference "#PWR046") (unit 1)
+          (reference "#PWR047") (unit 1)
         )
       )
@@
   (symbol (lib_id "Device:C") (at 155.575 132.715 0) (unit 1)
     (in_bom yes) (on_board yes) (dnp no) (fields_autoplaced)
-    (property "Reference" "C21" (at 159.385 131.445 0)
+    (property "Reference" "C22" (at 159.385 131.445 0)
       (effects (font (size 1.27 1.27)) (justify left))
     )
@@
       (project "Cable_Monitor"
         (path "/1f276d59-ad9b-4e70-a842-f3b7e562eb9b/de01ffac-1f9d-4a03-9ae5-48822ed64956"
-          (reference "C21") (unit 1)
+          (reference "C22") (unit 1)
         )
       )
@@
   (symbol (lib_id "Device:C") (at 103.505 106.68 90) (unit 1)
     (in_bom yes) (on_board yes) (dnp no) (fields_autoplaced)
-    (property "Reference" "C19" (at 103.505 99.06 90)
+    (property "Reference" "C20" (at 103.505 99.06 90)
       (effects (font (size 1.27 1.27)))
     )
@@
       (project "Cable_Monitor"
         (path "/1f276d59-ad9b-4e70-a842-f3b7e562eb9b/de01ffac-1f9d-4a03-9ae5-48822ed64956"
-          (reference "C19") (unit 1)
+          (reference "C20") (unit 1)
         )
       )
@@
   (symbol (lib_id "power:GND") (at 90.17 65.405 0) (unit 1)
     (in_bom yes) (on_board yes) (dnp no) (fields_autoplaced)
-    (property "Reference" "#PWR044" (at 90.17 71.755 0)
+    (property "Reference" "#PWR045" (at 90.17 71.755 0)
       (effects (font (size 1.27 1.27)) hide)
     )
@@
       (project "Cable_Monitor"
         (path "/1f276d59-ad9b-4e70-a842-f3b7e562eb9b/de01ffac-1f9d-4a03-9ae5-48822ed64956"
-          (reference "#PWR044") (unit 1)
+          (reference "#PWR045") (unit 1)
         )
       )
@@
   (symbol (lib_id "power:GND") (at 90.805 121.285 0) (unit 1)
     (in_bom yes) (on_board yes) (dnp no) (fields_autoplaced)
-    (property "Reference" "#PWR045" (at 90.805 127.635 0)
+    (property "Reference" "#PWR046" (at 90.805 127.635 0)
       (effects (font (size 1.27 1.27)) hide)
     )
@@
       (project "Cable_Monitor"
         (path "/1f276d59-ad9b-4e70-a842-f3b7e562eb9b/de01ffac-1f9d-4a03-9ae5-48822ed64956"
-          (reference "#PWR045") (unit 1)
+          (reference "#PWR046") (unit 1)
         )
       )
@@
   (symbol (lib_id "power:+3V0") (at 41.275 160.02 0) (unit 1)
     (in_bom yes) (on_board yes) (dnp no)
-    (property "Reference" "#PWR042" (at 41.275 163.83 0)
+    (property "Reference" "#PWR043" (at 41.275 163.83 0)
       (effects (font (size 1.27 1.27)) hide)
     )
@@
       (project "Cable_Monitor"
         (path "/1f276d59-ad9b-4e70-a842-f3b7e562eb9b/de01ffac-1f9d-4a03-9ae5-48822ed64956"
-          (reference "#PWR042") (unit 1)
-        )
-      )
+          (reference "#PWR043") (unit 1)
+        )
+      )
